File: Electronic/Designs/DAC/DAC.brd (EAGLE design)
At the start: 50 x 50 mm, 36 parts

Commit message: added new part to dac board
Parts:
- C5, C7: value 0.1uf -> 1uf
- JP1: value (none) -> PWR
- JP3: value (none) -> DIGITAL
- U$4: value OPA4227UA -> OPA2227UA; device OPAX22X:SOIC-14 -> OPAX22X:SOIC-8
- moved U$4 3.22 mm to (24.2, 5.89)
- renumbered JP4 to AOUT
Connections:
- new net V+: U$2.P$4
- new net V-: U$2.P$11
- net +15V: now also C4.1, U$4.P$8; no longer C5.1, U$2.P$4, U$4.P$4
- net -15V: now also C5.1, U$4.P$4; no longer C4.1, U$2.P$11, U$4.P$11
- net BIAS: now also U$4.P$7; no longer U$4.P$14
- net N$21: now also U$4.P$5; no longer U$4.P$12
- net N$22: now also U$4.P$6; no longer U$4.P$13
Routing:
- net +15V: track 9.88 -> 2.65 mm, vias 2 -> 0
- net -15V: track 6.76 -> 0.00 mm, vias 2 -> 0
- net N$21: track 9.52 -> 3.64 mm
- net B: track 22.6 -> 16.9 mm
- net +5V: track 6.36 -> 3.89 mm
- net N$22: track 5.03 -> 2.65 mm
- net N$19: track 5.14 -> 3.38 mm
- net BIAS: track 2.84 -> 1.89 mm
