File: Electronic/Designs/TunnelingAmp/TunnelingAmp.brd (EAGLE design)
At the start: 50 x 50 mm, 8 parts, among them U1 OPA627AUE4

Commit message: Added guard ring to tunneling current amp
Parts:
- moved U1 27.1 mm to (21.8, 7.16), turned to 270 degrees
- moved C1 24.1 mm to (10.2, 14.0)
- moved C2 24.1 mm to (10.2, 6.35)
- moved C3 24.1 mm to (14.0, 14.0)
- moved C4 24.1 mm to (14.0, 6.35)
- moved JP1 24.1 mm to (5.08, 10.2)
- moved JP2 20.5 mm to (28.5, 13.9), turned to 90 degrees
- moved R1 15.3 mm to (23.1, 12.6)
Routing:
- net N$6: track 0.00 -> 15.8 mm
- net V+: track 0.00 -> 9.70 mm
- net V-: track 0.00 -> 9.70 mm
- net GND: track 0.00 -> 9.05 mm, vias 0 -> 11
- net N$5: track 0.00 -> 5.31 mm
- added copper zone on layer 1, net GND
Other:
- board size 50 x 50 mm -> 35 x 20 mm

Commit message: Added to tunneling amp
Parts:
- JP1: value (none) -> pwr
- JP2: value (none) -> out
- moved C4 6.53 mm to (20.5, 6.17), turned to 180 degrees
- moved JP2 4.54 mm to (27.4, 18.3)
- moved R1 4.54 mm to (22.0, 17.0)
- moved U1 4.54 mm to (20.7, 11.6)
- moved C2 4.31 mm to (14.4, 5.65)
- moved C1 2.42 mm to (12.5, 13.2)
- moved JP1 2.42 mm to (7.38, 9.41)
- moved C3 2.42 mm to (16.3, 13.2)
Routing:
- net V+: track 9.70 -> 19.8 mm
- net V-: track 9.70 -> 12.3 mm
- net N$5: track 5.31 -> 5.98 mm
- net GND: vias 11 -> 13
- added copper zone on layer 16, net GND
Other:
- board size 35 x 20 mm -> 35 x 25 mm
