File: Electronic/Designs/DAC2/DAC2.brd (EAGLE design)
At the start: 50 x 50 mm, 15 parts

Commit message: Added new piezoDrive and holes for DAC2 and new lib OPA627
Changed lines of the file:
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@@
 <setting verticaltext="up"/>
 </settings>
-<grid distance="0.0500000001" unitdist="mm" unit="mm" style="lines" multiple="1" display="no" altdistance="0.025" altunitdist="inch" altunit="inch"/>
+<grid distance="0.1" unitdist="mm" unit="mm" style="lines" multiple="1" display="no" altdistance="0.025" altunitdist="inch" altunit="inch"/>
 <layers>
 <layer number="1" name="Top" color="4" fill="1" visible="yes" active="yes"/>
@@
 </element>
 <element name="U$3" library="REF02" package="SO8" value="REF02AU" x="33.78" y="19.4" smashed="yes" rot="R180">
-<attribute name="NAME" x="39.97" y="23.29" size="1.27" layer="25" rot="R180"/>
-<attribute name="VALUE" x="35.92" y="15.11" size="1.27" layer="25" rot="R180"/>
+<attribute name="NAME" x="33.67" y="15.54" size="1.27" layer="25" rot="R180"/>
 </element>
 </elements>
@@
 <wire x1="27.55" y1="27.59" x2="27.53" y2="27.61" width="0.254" layer="1"/>
 </signal>
+<signal name="N$1" airwireshidden="yes">
+<via x="3.5" y="46.5" extent="1-16" drill="2" diameter="6"/>
+<via x="46.5" y="46.5" extent="1-16" drill="2" diameter="6"/>
+<via x="46.5" y="3.5" extent="1-16" drill="2" diameter="6"/>
+<via x="3.5" y="3.5" extent="1-16" drill="2" diameter="6"/>
+<wire x1="3.5" y1="46.5" x2="46.5" y2="46.5" width="0" layer="19" extent="1-1"/>
+<wire x1="46.5" y1="3.5" x2="46.5" y2="46.5" width="0" layer="19" extent="1-1"/>
+<wire x1="3.5" y1="3.5" x2="3.5" y2="46.5" width="0" layer="19" extent="1-1"/>
+</signal>
 </signals>

Commit message: Added better Cmake QT Find and added dac2 piezo and tun boards
Parts:
- removed JP2: Output, pinhead:1X05
- added JP3: (no value), pinhead:1X06
Connections:
- net GND: now also JP3.1; no longer JP2.1
- net VOUTA: now also JP3.4; no longer JP2.4
- net VOUTB: now also JP3.3; no longer JP2.3
- net VOUTC: now also JP3.5; no longer JP2.5
- net VOUTD: now also JP3.2; no longer JP2.2
- net VREF: now also JP3.6
Routing:
- net VREF: track 11.0 -> 20.4 mm
- net VOUTD: track 11.7 -> 14.6 mm
- net VOUTC: track 9.53 -> 12.4 mm
- net VOUTB: track 12.2 -> 15.1 mm
- net VOUTA: track 11.6 -> 14.4 mm
Changed lines of the file:
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@@
 </element>
 <element name="JP1" library="pinhead" package="1X09" value="Input" x="11.88" y="32.91" rot="R90"/>
-<element name="JP2" library="pinhead" package="1X05" value="Output" x="35.07" y="34.12" rot="R270"/>
 <element name="U$1" library="DAC80004" package="TSSOP14" value="DAC80004IPW" x="26.23" y="30.41" rot="R90"/>
 <element name="U$2" library="TDA3664" package="SOT223" value="TDA3664/N1" x="22.38" y="11.68" smashed="yes" rot="R90">
@@
 <attribute name="NAME" x="33.67" y="15.54" size="1.27" layer="25" rot="R180"/>
 </element>
+<element name="JP3" library="pinhead" package="1X06" value="" x="37.7" y="32.6" rot="R270"/>
 </elements>
 <signals>
@@
 <wire x1="26.23" y1="29.48" x2="26.75" y2="29.95" width="0.254" layer="1"/>
 <wire x1="26.75" y1="29.95" x2="30.95" y2="29.95" width="0.4064" layer="1"/>
-<contactref element="JP2" pad="4"/>
 <wire x1="30.95" y1="29.95" x2="32.55" y2="31.55" width="0.4064" layer="1"/>
-<wire x1="32.55" y1="31.55" x2="35.04" y2="31.55" width="0.4064" layer="1"/>
-<wire x1="35.04" y1="31.55" x2="35.07" y2="31.58" width="0.4064" layer="1"/>
+<contactref element="JP3" pad="4"/>
+<wire x1="32.55" y1="31.55" x2="37.7" y2="31.55" width="0.4064" layer="1"/>
+<wire x1="37.7" y1="31.55" x2="37.7" y2="31.33" width="0.4064" layer="1"/>
 </signal>
 <signal name="VOUTB">
@@
 <wire x1="26.23" y1="31.42" x2="26.8" y2="30.85" width="0.254" layer="1"/>
 <wire x1="26.8" y1="30.85" x2="29.85" y2="30.85" width="0.4064" layer="1"/>
-<contactref element="JP2" pad="3"/>
 <wire x1="29.85" y1="30.85" x2="33.1" y2="34.1" width="0.4064" layer="1"/>
-<wire x1="33.1" y1="34.1" x2="35.05" y2="34.1" width="0.4064" layer="1"/>
-<wire x1="35.05" y1="34.1" x2="35.07" y2="34.12" width="0.4064" layer="1"/>
+<contactref element="JP3" pad="3"/>
+<wire x1="33.1" y1="34.1" x2="37.7" y2="34.1" width="0.4064" layer="1"/>
+<wire x1="37.7" y1="34.1" x2="37.7" y2="33.87" width="0.4064" layer="1"/>
 </signal>
 <signal name="VOUTC">
@@
 <wire x1="26.88" y1="27.61" x2="26.88" y2="28.88" width="0.254" layer="1"/>
 <wire x1="26.88" y1="28.88" x2="27.05" y2="29.05" width="0.254" layer="1"/>
-<wire x1="27.05" y1="29.05" x2="28.95" y2="29.05" width="0.4064" layer="1"/>
-<contactref element="JP2" pad="5"/>
-<wire x1="28.95" y1="29.05" x2="35.07" y2="29.04" width="0.4064" layer="1"/>
+<contactref element="JP3" pad="5"/>
+<wire x1="27.05" y1="29.05" x2="37.7" y2="29.05" width="0.4064" layer="1"/>
+<wire x1="37.7" y1="29.05" x2="37.7" y2="28.79" width="0.4064" layer="1"/>
 </signal>
 <signal name="VOUTD">
@@
 <wire x1="26.88" y1="31.92" x2="27.05" y2="31.75" width="0.254" layer="1"/>
 <wire x1="27.05" y1="31.75" x2="29" y2="31.75" width="0.4064" layer="1"/>
-<contactref element="JP2" pad="2"/>
 <wire x1="29" y1="31.75" x2="34" y2="36.75" width="0.4064" layer="1"/>
-<wire x1="34" y1="36.75" x2="34.98" y2="36.75" width="0.4064" layer="1"/>
-<wire x1="34.98" y1="36.75" x2="35.07" y2="36.66" width="0.4064" layer="1"/>
+<contactref element="JP3" pad="2"/>
+<wire x1="34" y1="36.75" x2="37.7" y2="36.75" width="0.4064" layer="1"/>
+<wire x1="37.7" y1="36.75" x2="37.7" y2="36.41" width="0.4064" layer="1"/>
 </signal>
 <signal name="VDD">
@@
 <vertex x="0" y="50"/>
 </polygon>
-<contactref element="JP2" pad="1"/>
 <contactref element="JP1" pad="9"/>
 <wire x1="25.58" y1="33.21" x2="25.58" y2="34.48" width="0.254" layer="1"/>
@@
 <wire x1="25.6" y1="34.5" x2="25.6" y2="31.95" width="0.254" layer="1"/>
 <wire x1="25.6" y1="31.95" x2="25.55" y2="31.9" width="0.254" layer="1"/>
+<contactref element="JP3" pad="1"/>
 </signal>
 <signal name="VREF">
@@
 <wire x1="29.5" y1="25.85" x2="29.68" y2="25.85" width="0.4064" layer="1"/>
 <wire x1="29.68" y1="25.85" x2="30.05" y2="25.48" width="0.4064" layer="1"/>
+<contactref element="JP3" pad="6"/>
+<wire x1="30.05" y1="25.48" x2="30.05" y2="26.65" width="0.4064" layer="1"/>
+<wire x1="30.05" y1="26.65" x2="30.5" y2="27.1" width="0.4064" layer="1"/>
+<wire x1="30.5" y1="27.1" x2="35.3" y2="27.1" width="0.4064" layer="1"/>
+<wire x1="35.3" y1="27.1" x2="36.1" y2="26.3" width="0.4064" layer="1"/>
+<wire x1="36.1" y1="26.3" x2="37.65" y2="26.3" width="0.4064" layer="1"/>
+<wire x1="37.65" y1="26.3" x2="37.7" y2="26.25" width="0.4064" layer="1"/>
 </signal>
 <signal name="VIN">

Commit message: added change to DAC2 board
Parts:
- JP3: value (none) -> Output
Changed lines of the file:
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@@
 <attribute name="NAME" x="33.67" y="15.54" size="1.27" layer="25" rot="R180"/>
 </element>
-<element name="JP3" library="pinhead" package="1X06" value="" x="37.7" y="32.6" rot="R270"/>
+<element name="JP3" library="pinhead" package="1X06" value="Output" x="37.7" y="32.6" rot="R270"/>
 </elements>
 <signals>
