File: Electronic/Designs/ADC/ADC.brd (EAGLE design)
At the start: 50 x 50 mm, 12 parts

Commit message: moved silkscreen text in ADC
Parts:
- C1: value 100nf -> 2.2uf
Changed lines of the file:
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@@
 </autorouter>
 <elements>
-<element name="C1" library="resistor" package="C0603" value="100nf" x="25.52" y="15.92" smashed="yes" rot="R90">
+<element name="C1" library="resistor" package="C0603" value="2.2uf" x="25.52" y="15.92" smashed="yes" rot="R90">
 <attribute name="NAME" x="24.185" y="14.035" size="1.27" layer="25" rot="R90"/>
 <attribute name="VALUE" x="26.125" y="9.035" size="1.27" layer="27" rot="R90"/>
